File: piano-tiles-pcb/piano-tiles-pcb.kicad_sch (KiCad schematic)
At the start: 19 parts, among them IC2 MSPM0G3507SPTR, J1 Conn_01x05, J2 Conn_01x05, SW1 SW_SPST, SW2 SW_SPST, SW3 SW_SPST, SW4 SW_SPST, SW5 SW_SPDT

Commit message: first order
Parts:
- removed BT1: Battery_Cell, Battery:BatteryHolder_Keystone_1060_1x2032, symbol Device:Battery_Cell
- removed C3: 100uF, Capacitor_SMD:C_1206_3216Metric, symbol Device:C
- removed SW5: SW_SPDT, ELEC327-Kicad:SW_EG1270, symbol Switch:SW_SPDT
- added J3: Barrel_Jack_MountingPin, Connector_BarrelJack:BarrelJack_CUI_PJ-063AH_Horizontal, symbol Connector:Barrel_Jack_MountingPin
- added SW6: SW_SPDT, ELEC327-Kicad:SW_EG1270, symbol Switch:SW_SPDT
- C1: footprint Capacitor_SMD:C_0603_1608Metric -> Capacitor_SMD:C_1206_3216Metric_Pad1.33x1.80mm_HandSolder; LCSC Part # C19702 -> (none)
- C2: footprint Capacitor_SMD:C_0603_1608Metric_Pad1.08x0.95mm_HandSolder -> Capacitor_SMD:C_1206_3216Metric_Pad1.33x1.80mm_HandSolder; LCSC Part # C1591 -> (none)
- C4: footprint Capacitor_SMD:C_0805_2012Metric -> Capacitor_SMD:C_1206_3216Metric_Pad1.33x1.80mm_HandSolder
- C6: footprint Capacitor_SMD:C_0402_1005Metric -> Capacitor_SMD:C_1206_3216Metric_Pad1.33x1.80mm_HandSolder
- MSPM0G3507_Breakout1: footprint Connector_PinHeader_2.54mm:PinHeader_2x16_P2.54mm_Vertical -> ELEC327-Kicad:QFN32Breakout-PinHeader_2x16_P2.54mm_Vertical
- R5: footprint Resistor_SMD:R_0603_1608Metric -> Resistor_SMD:R_1206_3216Metric_Pad1.30x1.75mm_HandSolder
- R6: footprint Resistor_SMD:R_0402_1005Metric -> Resistor_SMD:R_1206_3216Metric_Pad1.30x1.75mm_HandSolder
- SW1, SW2, SW3, SW4: footprint Button_Switch_SMD:SW_SPST_PTS647_Sx38 -> Button_Switch_THT:SW_PUSH_6mm_H5mm; LCSC Part # C2799279 -> (none); MPN C2799279 -> (none)
Connections:
- net BUTTON1_IO: now also J1.1 (Pin_1), MSPM0G3507_Breakout1.30 (Pin_30); no longer J1.5 (Pin_5), MSPM0G3507_Breakout1.27 (Pin_27)
- net BUTTON2_IO: now also J1.2 (Pin_2), MSPM0G3507_Breakout1.29 (Pin_29); no longer J1.4 (Pin_4), MSPM0G3507_Breakout1.28 (Pin_28)
- net BUTTON3_IO: now also MSPM0G3507_Breakout1.28 (Pin_28); no longer MSPM0G3507_Breakout1.29 (Pin_29)
- net BUTTON4_IO: now also J1.4 (Pin_4), MSPM0G3507_Breakout1.27 (Pin_27); no longer J1.2 (Pin_2), MSPM0G3507_Breakout1.30 (Pin_30)
- net GND: now also J1.5 (Pin_5), J3.2; no longer J1.1 (Pin_1)
- net SWCLK: now also MSPM0G3507_Breakout1.24 (Pin_24)
- net SWDIO: now also MSPM0G3507_Breakout1.23 (Pin_23)
- net VDD: now also SW6.1 (A)
- net ACC_INT: no longer names the net of IC2.27 (PA12_/_FCC_IN)
- net ACC_INT: no longer MSPM0G3507_Breakout1.16 (Pin_16)
- new net: J3.1, SW6.2 (B)
Other:
- note added: "Power Smoothing"
- note removed: "Q. PA12 ACC_INT needed???"
- note removed: "Q: Cable plug instead of battery???"
- moved on the sheet: BZ1, C4, J2, MSPM0G3507_Breakout1, R6
